Commit message: ajout de projet ros2_nav2_slam

File: my_pkg/description/camera.xacro (robot description, xacro)
@@ -62,5 +62,5 @@
       <update_rate>20</update_rate>
       <topic>camera/image</topic>
-      <gz_frame_id>camera_link</gz_frame_id>
+      <frame_id>camera_link</frame_id>
     </sensor>
   </gazebo>

File: my_pkg/description/controle_gazebo.xacro (robot description, xacro)
@@ -22,5 +22,5 @@
             <publish_odom>true</publish_odom>
             <publish_odom_tf>true</publish_odom_tf>
-            <publish_wheel_tf>false</publish_wheel_tf>
+            <publish_wheel_tf>true</publish_wheel_tf>
            <!-- Pour publier la pose et la vitesse de mon robot sur nav_msgs/odometiee -->
             <odom_topic>odom</odom_topic>

File: my_pkg/description/gps.xacro (robot description, xacro)
@@ -13,5 +13,5 @@
         <update_rate>1</update_rate>
         <topic>navsat</topic>
-        <gz_frame_id>navsat_link</gz_frame_id>
+        <frame_id>navsat_link</frame_id>
         </sensor>
     </gazebo>

File: my_pkg/description/imu.xacro (robot description, xacro)
@@ -16,5 +16,5 @@
             <topic>imu</topic>
             <enable_metrics>true</enable_metrics>
-            <gz_frame_id>imu_link</gz_frame_id>
+            <frame_id>imu_link</frame_id>
         </sensor>
     </gazebo>

File: my_pkg/description/lidar.xacro (robot description, xacro)
@@ -1,8 +1,8 @@
 <?xml version="1.0"?>
-<robot xmlns:xacro="http://www.ros.org/wiki/xacro">
+<robot xmlns:xacro="http://www.ros.org/wiki/xacro" >
     <joint name="laser_joint" type="fixed">
         <parent link="chassis"/>
         <child link="laser_frame"/>
-        <origin xyz="0.06 0 0.125" rpy="0 0 0"/>
+        <origin xyz="0.122 0 0.180" rpy="0 0 0"/>
     </joint>
     <link name="laser_frame">
@@ -10,4 +10,11 @@
             <geometry>
                 <cylinder radius="0.05" length="0.04"/>
+            </geometry>
+            <material name="black"/>
+        </visual>
+        <visual>
+            <origin xyz="0 0 -0.05"/>
+            <geometry>
+                <cylinder radius="0.01" length="0.1"/>
             </geometry>
             <material name="black"/>
@@ -23,37 +30,33 @@
     </link>
     <gazebo reference="laser_frame">
-            <sensor name='laser' type='gpu_lidar'>
-                <pose>0 0 0 0 0 0</pose>
-                <topic>scan</topic>
-                <gz_frame_id>laser_frame</gz_frame_id>
-                <update_rate>10</update_rate>
-                <lidar>
-                    <scan>
-                        <horizontal>
-                            <samples>360</samples>
-                            <resolution>1</resolution>
-                            <min_angle>-1.57</min_angle>
-                            <max_angle>1.57</max_angle>
-                        </horizontal>
-                        <vertical>
-                            <samples>1</samples>
-                            <resolution>1</resolution>
-                            <min_angle>0.0</min_angle>
-                            <max_angle>0.0</max_angle>
-                        </vertical>
-                    </scan>
-                    <range>
-                            <min>0.08</min>
-                            <max>15.0</max>
-                            <resolution>0.01</resolution>
-                    </range>
-                    <!-- <noise>
-                        <type>gaussian</type>
-                        <mean>0.0</mean>
-                        <stddev>0.01</stddev>
-                    </noise> -->
-                </lidar>
-                <topic>scan</topic>
-            </sensor>
+        <material>Gazebo/Black</material>
+        <sensor name='laser' type='gpu_lidar'>
+            <pose>0 0 0 0 0 0</pose>
+            <topic>/scan</topic>
+            <frame_id>laser_frame</frame_id>
+            <update_rate>10</update_rate>
+            <lidar>
+              <scan>
+                <horizontal>
+                  <samples>640</samples>
+                  <resolution>1</resolution>
+                  <min_angle>-1.57</min_angle>
+                  <max_angle>1.57</max_angle>
+                </horizontal>
+                <vertical>
+                  <samples>1</samples>
+                  <resolution>1</resolution>
+                  <min_angle>0.0</min_angle>
+                  <max_angle>0.0</max_angle>
+                </vertical>
+              </scan>
+              <range>
+                <min>0.08</min>
+                <max>15.0</max>
+                <resolution>0.01</resolution>
+              </range>
+            </lidar>
+            <visualize>true</visualize>
+          </sensor>
     </gazebo>
 </robot>
