Commit message: configuratin de ros2_control et de la pile Nav2

File: my_pkg/description/camera.xacro (robot description, xacro)
@@ -1,67 +1,62 @@
 <?xml version="1.0"?>
-<robot xmlns:xacro="http://www.ros.org/wiki/xacro">
-    <!-- Le lien de la caméra -->
-      <!-- STEP 7 - Camera -->
-  <joint type="fixed" name="camera_joint">
-    <origin xyz="0.315 0 0.075" rpy="0 0 0"/>
-    <child link="camera_link"/>
-    <parent link="chassis"/>
-    <axis xyz="0 1 0" />
-  </joint>
-  <link name='camera_link'>
-    <pose>0 0 0 0 0 0</pose>
-    <inertial>
-      <mass value="0.1"/>
-      <origin xyz="0 0 0" rpy="0 0 0"/>
-      <inertia
-          ixx="1e-6" ixy="0" ixz="0"
-          iyy="1e-6" iyz="0"
-          izz="1e-6"
-      />
-    </inertial>
-    <collision name='collision'>
-      <origin xyz="0 0 0" rpy="0 0 0"/>
-      <geometry>
-        <box size=".03 .03 .03"/>
-      </geometry>
-    </collision>
-    <visual name='camera_link_visual'>
-      <origin xyz="0 0 0" rpy="0 0 0"/>
-      <geometry>
-        <box size=".03 .03 .03"/>
-      </geometry>
-    </visual>
-  </link>
-  <gazebo reference="camera_link">
-    <material>Gazebo/Red</material>
-  </gazebo>
-  <joint type="fixed" name="camera_optical_joint">
-    <origin xyz="0 0 0" rpy="-1.5707 0 -1.5707"/>
-    <child link="camera_link_optical"/>
-    <parent link="camera_link"/>
-  </joint>
-  <link name="camera_link_optical">
-  </link>
-    <!-- Plugin Gazebo pour simuler la caméra -->
-  <gazebo reference="camera_link">
-    <sensor name="wideangle_camera" type="wideanglecamera">
-      <camera>
-        <horizontal_fov>3.14</horizontal_fov>
-        <image>
-          <width>640</width>
-          <height>480</height>
-        </image>
-        <clip>
-          <near>0.1</near>
-          <far>15</far>
-        </clip>
-        <optical_frame_id>camera_link_optical</optical_frame_id>
-        <camera_info_topic>camera/camera_info</camera_info_topic>
-      </camera>
-      <always_on>1</always_on>
-      <update_rate>20</update_rate>
-      <topic>camera/image</topic>
-      <frame_id>camera_link</frame_id>
-    </sensor>
-  </gazebo>
+<robot xmlns:xacro="http://www.ros.org/wiki/xacro" >
+    <joint name="camera_joint" type="fixed">
+        <parent link="chassis"/>
+        <child link="camera_link"/>
+        <origin xyz="0.142 0 0.161" rpy="0 0 0"/>
+    </joint>
+    <link name="camera_link">
+        <visual>
+            <geometry>
+                <box size="0.010 0.03 0.03"/>
+            </geometry>
+            <material name="black"/>
+        </visual>
+        <visual>
+            <origin xyz="0 0 -0.05"/>
+            <geometry>
+                <cylinder radius="0.002" length="0.1"/>
+            </geometry>
+            <material name="black"/>
+        </visual>
+    </link>
+    <joint name="camera_optical_joint" type="fixed">
+        <parent link="camera_link"/>
+        <child link="camera_link_optical"/>
+        <origin xyz="0 0 0" rpy="${-pi/2} 0 ${-pi/2}"/>
+    </joint>
+    <link name="camera_link_optical"></link>
+    <gazebo reference="camera_link">
+        <material>Gazebo/Black</material>
+        <sensor name="rgbd_camera" type="rgbd_camera">
+            <update_rate>20</update_rate>
+            <topic>/image/image_raw</topic>
+            <gz_frame_id>camera_link_optical</gz_frame_id>
+            <camera>
+                <horizontal_fov>1.089</horizontal_fov>
+                <image>
+                    <width>640</width>
+                    <height>480</height>
+                    <format>RGB_INT8</format>
+                </image>
+                <clip>
+                    <near>0.05</near>
+                    <far>10.0</far>
+                </clip>
+            </camera>
+            <depth_camera>
+                <clip>
+                    <near>0.05</near>
+                    <far>10.0</far>
+                </clip>
+                <noise>
+                    <type>gaussian</type>
+                    <mean>0.0</mean>
+                    <stddev>0.001</stddev>
+                </noise>
+            </depth_camera>
+            <always_on>1</always_on>
+            <visualize>true</visualize>
+        </sensor>
+    </gazebo>
 </robot>

File: my_pkg/description/controle_gazebo.xacro (robot description, xacro)
@@ -1,42 +1,22 @@
-<?xml version = "1.0" ?>
-<robot xmlns:xacro="http://www.ros.org/wiki/xacro" >
-    <gazebo>
-         <plugin filename="gz-sim-diff-drive-system" name="gz::sim::systems::DiffDrive">
-            <odom_publisher_frequency>50</odom_publisher_frequency>
-            <left_joint>wheel_left_joint</left_joint>
-            <right_joint>wheel_right_joint</right_joint>
-            <wheel_separation>0.3</wheel_separation>
-            <wheel_diameter>0.1</wheel_diameter>
-            <max_wheel_torque>200</max_wheel_torque>
-            <max_wheel_acceleration>10.0</max_wheel_acceleration>
-            <!-- <max_velocity>3.0</max_velocity>
-            <max_linear_acceleration>1</max_linear_acceleration>
-            <min_linear_acceleration>-1</min_linear_acceleration>
-            <max_angular_acceleration>2</max_angular_acceleration>
-            <min_angular_acceleration>-2</min_angular_acceleration>
-            <max_linear_velocity>0.5</max_linear_velocity>
-            <min_linear_velocity>-0.5</min_linear_velocity>
-            <max_angular_velocity>1</max_angular_velocity>
-            <min_angular_velocity>-1</min_angular_velocity> -->
-            <topic>cmd_vel</topic>
-            <publish_odom>true</publish_odom>
-            <publish_odom_tf>true</publish_odom_tf>
-            <publish_wheel_tf>true</publish_wheel_tf>
-           <!-- Pour publier la pose et la vitesse de mon robot sur nav_msgs/odometiee -->
-            <odom_topic>odom</odom_topic>
-<!-- Pour pour publier la transformation odom==>base_link  -->
-            <tf_topic>tf</tf_topic>
-            <frame_id>odom</frame_id>
-            <child_frame_id>base_link</child_frame_id>
-            <!-- <odometry_frame>odom</odometry_frame>
-            <robot_base_frame>base_link</robot_base_frame> -->
-         </plugin>
-         <!-- <plugin
-            filename="gz-sim-joint-state-publisher-system"
-            name="gz::sim::systems::JointStatePublisher">
-            <topic>joint_states</topic>
-            <joint_name>wheel_left_joint</joint_name>
-            <joint_name>wheel_right_joint</joint_name>
-         </plugin> -->
-    </gazebo>
+<?xml version="1.0"?>
+<robot xmlns:xacro="http://www.ros.org/wiki/xacro">
+<gazebo>
+    <plugin name="gz::sim::systems::DiffDrive" filename="gz-sim-diff-drive-system">
+      <left_joint>front_left_wheel_joint</left_joint>
+      <left_joint>rear_left_wheel_joint</left_joint>
+      <right_joint>front_right_wheel_joint</right_joint>
+      <right_joint>rear_right_wheel_joint</right_joint>
+      <!-- Paramètres -->
+      <wheel_separation>${wheel_offset_y * 2}</wheel_separation>
+      <wheel_radius>${wheel_radius}</wheel_radius>
+      <topic>/cmd_vel</topic>
+      <max_linear_acceleration>0.33</max_linear_acceleration>
+      <frame_id>odom</frame_id>
+      <child_frame_id>base_footprint</child_frame_id>
+      <odom_topic>/wheel_odom</odom_topic>
+      <odom_publisher_frequency>30</odom_publisher_frequency>
+      <odom_publish_tf>false</odom_publish_tf>
+      <!--<tf_topic>/tf</tf_topic> -->
+    </plugin>
+  </gazebo>
 </robot>

File: my_pkg/description/gps.xacro (robot description, xacro)
@@ -1,18 +1,45 @@
-<?xml version="1.0" ?>
+<?xml version="1.0"?>
 <robot xmlns:xacro="http://www.ros.org/wiki/xacro">
-    <joint name="navsat_joint" type="fixed">
-        <origin xyz="0 0 0" rpy="0 0 0" />
-        <parent link="chassis"/>
-        <child link="navsat_link" />
-    </joint>
-    <link name="navsat_link">
-    </link>
-    <gazebo reference="navsat_link">
-        <sensor name="navsat" type="navsat">
-        <always_on>1</always_on>
-        <update_rate>1</update_rate>
-        <topic>navsat</topic>
-        <frame_id>navsat_link</frame_id>
-        </sensor>
-    </gazebo>
+  <!-- Joint fixe entre le châssis et le GNSS -->
+  <joint name="gnss_joint" type="fixed">
+    <parent link="chassis"/>
+    <child link="gnss_frame"/>
+    <origin xyz="0.10 0 0.80" rpy="0 0 0"/>
+  </joint>
+  <link name="gnss_frame">
+  </link>
+  <!-- Définition du capteur GNSS pour Gazebo Sim -->
+  <gazebo reference="gnss_frame">
+    <material>Gazebo/Black</material>
+    <!-- Capteur GNSS -->
+    <sensor name="gnss" type="navsat">
+      <pose>0 0 0 0 0 0</pose>
+      <topic>/gnss/fix</topic>
+      <gz_frame_id>gnss_frame</gz_frame_id>
+      <update_rate>10</update_rate>
+      <navsat>
+        <position_sensing>
+          <horizontal>
+            <noise type="gaussian">
+              <mean>0.0</mean>
+              <stddev>0.5</stddev>
+            </noise>
+          </horizontal>
+          <vertical>
+            <noise type="gaussian">
+              <mean>0.0</mean>
+              <stddev>1.0</stddev>
+            </noise>
+          </vertical>
+        </position_sensing>
+        <velocity_sensing>
+          <noise type="gaussian">
+            <mean>0.0</mean>
+            <stddev>0.1</stddev>
+          </noise>
+        </velocity_sensing>
+      </navsat>
+      <visualize>true</visualize>
+    </sensor>
+  </gazebo>
 </robot>

File: my_pkg/description/imu.xacro (robot description, xacro)
@@ -1,2 +1,3 @@
+<!--
 <?xml version="1.0"?>
 <robot xmlns:xacro="http://www.ros.org/wiki/xacro">
@@ -8,5 +9,5 @@
     <link name="imu_link">
     </link>
-  <!-- Le pluging de l'imu -->
+  <! Le pluging de l'imu >  commentaire
     <gazebo reference= 'imu_link'>
         <sensor name=' imu' type='imu'>
@@ -19,3 +20,82 @@
         </sensor>
     </gazebo>
+</robot>   -->
+<?xml version="1.0"?>
+<robot xmlns:xacro="http://www.ros.org/wiki/xacro" >
+<joint name="imu_joint" type="fixed">
+    <parent link="chassis"/>
+    <child link="imu_link"/>
+    <origin xyz="0 0 ${chassis_height/2}" rpy="0 0 0"/>
+  </joint>
+ <link name="imu_link">
+<!-- le imu est invisible
+  <visual>
+    <geometry>
+      <box size="0.05 0.05 0.05"/>
+    </geometry>
+  </visual>
+  <collision>
+    <geometry>
+      <box size="0 0.05 0.05"/>
+    </geometry>
+  </collision>
+  <inertial>
+            <mass value="0.1" />
+            <inertia ixx="0.01" ixy="0.0" ixz="0"
+            iyy="0.01" iyz="0" izz="0.01" />
+  </inertial> -->
+</link>
+<gazebo reference="imu_link">
+  <!-- <material>Gazebo/Black</material> -->
+  <sensor name="imu_sensor" type="imu">
+    <always_on>true</always_on>
+    <update_rate>200</update_rate>
+    <gz_frame_id>imu_link</gz_frame_id>
+    <topic>/imu</topic>
+    <imu>
+      <orientation_reference_frame parent_frame="imu_link" custom_rpy="0 0 0"/>
+      <angular_velocity>
+        <x>
+          <noise type="gaussian">
+            <mean>0.0</mean>
+            <stddev>2e-4</stddev>
+          </noise>
+        </x>
+        <y>
+          <noise type="gaussian">
+            <mean>0.0</mean>
+            <stddev>2e-4</stddev>
+          </noise>
+        </y>
+        <z>
+          <noise type="gaussian">
+            <mean>0.0</mean>
+            <stddev>2e-4</stddev>
+          </noise>
+        </z>
+      </angular_velocity>
+      <linear_acceleration>
+        <x>
+          <noise type="gaussian">
+            <mean>0.0</mean>
+            <stddev>1.7e-2</stddev>
+          </noise>
+        </x>
+        <y>
+          <noise type="gaussian">
+            <mean>0.0</mean>
+            <stddev>1.7e-2</stddev>
+          </noise>
+        </y>
+        <z>
+          <noise type="gaussian">
+            <mean>0.0</mean>
+            <stddev>1.7e-2</stddev>
+          </noise>
+        </z>
+      </linear_acceleration>
+        <orientation_enabled>true</orientation_enabled>
+      </imu>
+    </sensor>
+  </gazebo>
 </robot>

File: my_pkg/description/lidar.xacro (robot description, xacro)
@@ -4,5 +4,5 @@
         <parent link="chassis"/>
         <child link="laser_frame"/>
-        <origin xyz="0.122 0 0.180" rpy="0 0 0"/>
+        <origin xyz="0.122 0 0.212" rpy="0 0 0"/>
     </joint>
     <link name="laser_frame">
@@ -34,5 +34,5 @@
             <pose>0 0 0 0 0 0</pose>
             <topic>/scan</topic>
-            <frame_id>laser_frame</frame_id>
+            <gz_frame_id>laser_frame</gz_frame_id>
             <update_rate>10</update_rate>
             <lidar>
@@ -41,6 +41,6 @@
                   <samples>640</samples>
                   <resolution>1</resolution>
-                  <min_angle>-1.57</min_angle>
-                  <max_angle>1.57</max_angle>
+                  <min_angle>-3.14</min_angle>
+                  <max_angle>3.14</max_angle>
                 </horizontal>
                 <vertical>
@@ -53,5 +53,5 @@
               <range>
                 <min>0.08</min>
-                <max>15.0</max>
+                <max>10.0</max>
                 <resolution>0.01</resolution>
               </range>
@@ -61,2 +61,62 @@
     </gazebo>
 </robot>
+<!--
+<?xml version="1.0"?>
+<robot xmlns:xacro="http://www.ros.org/wiki/xacro">
+    <joint name="laser_joint" type="fixed">
+        <parent link="chassis"/>
+        <child link="laser_frame"/>
+        <origin xyz="0.06 0 0.125" rpy="0 0 0"/>
+    </joint>
+    <link name="laser_frame">
+        <visual>
+            <geometry>
+                <cylinder radius="0.05" length="0.04"/>
+            </geometry>
+            <material name="black"/>
+        </visual>
+        <collision>
+            <geometry>
+                <cylinder radius="0.05" length="0.04"/>
+            </geometry>
+        </collision>
+        <xacro:inertial_cylinder mass="0.1" length="0.04" radius="0.05">
+            <origin xyz="0 0 0" rpy="0 0 0"/>
+        </xacro:inertial_cylinder>
+    </link>
+    <gazebo reference="laser_frame">
+            <sensor name='laser' type='gpu_lidar'>
+                <pose>0 0 0 0 0 0</pose>
+                <topic>/scan</topic>
+                <gz_frame_id>laser_frame</gz_frame_id>
+                <update_rate>10</update_rate>
+                <lidar>
+                    <scan>
+                        <horizontal>
+                            <samples>640</samples>
+                            <resolution>1</resolution>
+                            <min_angle>-1.57</min_angle>
+                            <max_angle>1.57</max_angle>
+                        </horizontal>
+                        <vertical>
+                            <samples>1</samples>
+                            <resolution>1</resolution>
+                            <min_angle>0.0</min_angle>
+                            <max_angle>0.0</max_angle>
+                        </vertical>
+                    </scan>
+                    <range>
+                            <min>0.8</min>
+                            <max>15.0</max>
+                            <resolution>0.01</resolution>
+                    </range>
+                   - <noise>
+                        <type>gaussian</type>
+                        <mean>0.0</mean>
+                        <stddev>0.01</stddev>
+                    </noise>
+                </lidar>
+            </sensor>
+    </gazebo>
+</robot>
+-->

File: my_pkg/description/robot.urdf.xacro (robot description, xacro)
@@ -1,14 +1,24 @@
+<?xml version="1.0"?>
+<robot xmlns:xacro="http://www.ros.org/wiki/xacro"  name="my_robot">
+    <xacro:include filename="robot.xacro"  />
+    <xacro:include filename="lidar.xacro" />
+    <xacro:include filename="camera.xacro" />
+     <xacro:include filename="gps.xacro" />
+     <xacro:include filename="odom.xacro" />
+      <xacro:include filename="ros2_control.xacro" />
+    <xacro:include filename="controle_gazebo.xacro" />
+     <!-- Imu -->
+     <xacro:include filename='imu.xacro'/>
+</robot>
+<!--
 <?xml  version ="1.0" ?>
 <robot  name="my_robot" xmlns:xacro="http://www.ros.org/wiki/xacro">
      <xacro:include filename="robot.xacro" />
-     <!--Inclure le lidar -->
      <xacro:include filename="lidar.xacro"/>
-     <!--Control robot-->
+     Control robot
      <xacro:include filename = "controle_gazebo.xacro"/>
-          <!-- camera -->
      <xacro:include filename='camera.xacro' />
-           <!-- Imu -->
      <xacro:include filename='imu.xacro'/>
-     <!-- Navsat -->
      <xacro:include filename="gps.xacro"/>
 </robot>
+-->
