Commit message: configuratin de ros2_control et de la pile Nav2

File: my_pkg/description/robot.xacro (robot description, xacro)
@@ -1,13 +1,21 @@
 <?xml version="1.0"?>
 <robot xmlns:xacro="http://www.ros.org/wiki/xacro">
-    <!-- Inclusion des macros d'inertie -->
-    <xacro:include filename="inertial.xacro"/>
-    <!-- Dimensions du châssis -->
-    <xacro:property name="chassis_length" value="0.3"/>
-    <xacro:property name="chassis_width" value="0.2"/>
-    <xacro:property name="chassis_height" value="0.1"/>
-    <!-- Matériaux -->
+    <xacro:include filename="inertial_macros.xacro" />
+    <!-- CHASSIS  CONF-->
+    <xacro:property name="chassis_length" value="0.335"/>
+    <xacro:property name="chassis_width" value="0.265"/>
+    <xacro:property name="chassis_height" value="0.138"/>
+    <xacro:property name="chassis_mass" value="1.5"/>
+    <!--  ROUES CONF -->
+    <xacro:property name="wheel_radius" value="0.06"/>
+    <xacro:property name="wheel_thickness" value="0.026"/>
+    <xacro:property name="wheel_mass" value="0.09"/>
+    <xacro:property name="wheel_offset_z" value="0.01"/>
+    <!-- POSITIONS DES ROUES  -->
+    <xacro:property name="wheel_offset_x_front" value="0.120"/>
+    <xacro:property name="wheel_offset_x_rear" value="-0.120"/>
+    <xacro:property name="wheel_offset_y" value="0.1485"/>
     <material name="white">
-        <color rgba="1 1 1 1"/>
+        <color rgba="1 1 1 1" />
     </material>
     <material name="orange">
@@ -23,143 +31,66 @@
         <color rgba="1 0 0 1"/>
     </material>
-    <!-- Chassis -->
+    <link name="base_link">
+    </link>
+    <joint name="base_footprint_joint" type="fixed">
+        <parent link="base_footprint"/>
+        <child link="base_link"/>
+        <origin xyz="0 0 ${wheel_radius}" rpy="0 0 0"/>
+    </joint>
+    <link name="base_footprint">
+    </link>
+    <joint name="chassis_joint" type="fixed">
+        <parent link="base_link"/>
+        <child link="chassis"/>
+        <origin xyz="0 0 ${-wheel_offset_z}"/>
+    </joint>
     <link name="chassis">
         <visual>
-            <origin xyz="${chassis_length/2} 0 ${chassis_height/2}"/>
+            <origin xyz="0 0 ${chassis_height/2}"/>
             <geometry>
                 <box size="${chassis_length} ${chassis_width} ${chassis_height}"/>
             </geometry>
-            <material name="white"/>
+            <material name="orange"/>
         </visual>
         <collision>
-            <origin xyz="${chassis_length/2} 0 ${chassis_height/2}"/>
+            <origin xyz="0 0 ${chassis_height/2}"/>
             <geometry>
                 <box size="${chassis_length} ${chassis_width} ${chassis_height}"/>
             </geometry>
         </collision>
-        <xacro:inertial_box mass="0.5" x="${chassis_length}" y="${chassis_width}" z="${chassis_height}">
-            <origin xyz="${chassis_length/2} 0 ${chassis_height/2}" rpy="0 0 0"/>
+        <xacro:inertial_box mass="${chassis_mass}" x="${chassis_length}" y="${chassis_width}" z="${chassis_height}">
+            <origin xyz="0 0 ${chassis_height/2}" rpy="0 0 0"/>
         </xacro:inertial_box>
     </link>
-    <!-- Base link -->
-    <link name="base_link"/>
-    <!-- BASE_FOOTPRINT LINK -->
-    <joint name="base_footprint_joint" type="fixed">
-        <parent link="base_link"/>
-        <child link="base_footprint"/>
-        <origin xyz="0 0 0" rpy="0 0 0"/>
-    </joint>
-    <link name="base_footprint">
-    </link>
-     <!-- Roue gauche -->
-    <joint name="base_link_joint" type="fixed">
-        <parent link="base_link"/>
-        <child link="chassis"/>
-        <origin xyz="-0.1 0 0" rpy="0 0 0"/>
-    </joint>
-    <gazebo reference="chassis">
-        <material>Gazebo/White</material>
-    </gazebo>
-    <link name="wheel_left">
-        <visual>
-            <origin xyz="0 0 0" rpy="0 0 0"/>
-            <geometry>
-                <cylinder length="0.04" radius="0.05"/>
-            </geometry>
-            <material name="blue"/>
-        </visual>
-        <collision>
-            <origin xyz="0 0 0" rpy="0 0 0"/>
-            <geometry>
-                <cylinder length="0.04" radius="0.05"/>
-            </geometry>
-        </collision>
-        <xacro:inertial_cylinder mass="0.1" length="0.04" radius="0.05">
-            <origin xyz="0 0 0" rpy="0 0 0"/>
-        </xacro:inertial_cylinder>
-    </link>
-    <gazebo reference="wheel_left">
-        <material>Gazebo/Blue</material>
-        <mu1>0.2</mu1>
-        <mu2>0.2</mu2>
-        <kp>1000000.0</kp>
-        <kd>100.0</kd>
-        <minDepth>0.0001</minDepth>
-        <maxVel>1.0</maxVel>
-    </gazebo>
-    <joint name="wheel_left_joint" type="continuous">
-        <parent link="base_link"/>
-        <child link="wheel_left"/>
-        <origin xyz="0 ${chassis_width/2 + 0.03} 0" rpy="-1.57 0 0"/>
-        <axis xyz="0 0 1"/>
-    </joint>
-    <!-- Roue droite -->
-    <link name="wheel_right">
-        <visual>
-            <origin xyz="0 0 0" rpy="0 0 0"/>
-            <geometry>
-                <cylinder length="0.04" radius="0.05"/>
-            </geometry>
-            <material name="blue"/>
-        </visual>
-        <collision>
-            <origin xyz="0 0 0" rpy="0 0 0"/>
-            <geometry>
-                <cylinder length="0.04" radius="0.05"/>
-            </geometry>
-        </collision>
-        <xacro:inertial_cylinder mass="0.1" length="0.04" radius="0.05">
-            <origin xyz="0 0 0" rpy="0 0 0"/>
-        </xacro:inertial_cylinder>
-    </link>
-    <gazebo reference="wheel_right">
-        <material>Gazebo/Blue</material>
-        <mu1>0.2</mu1>
-        <mu2>0.2</mu2>
-        <kp>1000000.0</kp>
-        <kd>100.0</kd>
-        <minDepth>0.0001</minDepth>
-        <maxVel>1.0</maxVel>
-    </gazebo>
-    <joint name="wheel_right_joint" type="continuous">
-        <parent link="base_link"/>
-        <child link="wheel_right"/>
-        <origin xyz="0 -${chassis_width/2 + 0.03} 0" rpy="1.57 0 0"/>
-        <axis xyz="0 0 -1"/>
-    </joint>
-    <!-- Roue folle (caster) -->
-    <link name="caster_wheel">
-        <visual>
-            <geometry>
-                <sphere radius="0.05"/>
-            </geometry>
-            <origin xyz="0 0 0" rpy="0 0 0"/>
-            <material name="black">
-            </material>
-        </visual>
-        <collision>
-            <geometry>
-                <sphere radius="0.05"/>
-                <surface><friction><ode>
-                    <mu>0.001</mu>
-                    <mu2>0.001</mu2>
-                </ode></friction></surface>
-            </geometry>
-            <origin xyz="0 0 0" rpy="0 0 0"/>
-            <material name="black"/>
-        </collision>
-        <xacro:inertial_sphere mass="0.1" radius="0.05">
-            <origin xyz="0 0 0" rpy="0 0 0"/>
-        </xacro:inertial_sphere>
-    </link>
-    <joint name="caster_wheel_joint" type="fixed">
-        <parent link="chassis"/>
-        <child link="caster_wheel"/>
-        <origin xyz="0.24 0 0" rpy="0 0 0"/>
-    </joint>
-    <gazebo reference="caster_wheel">
-        <material>Gazebo/Black</material>
-        <mu1 value="0.001"/>
-        <mu2 value="0.001"/>
-    </gazebo>
+    <!-- MACRO POUR CRÉER UNE ROUE -->
+    <xacro:macro name="wheel" params="prefix x_pos y_pos">
+        <joint name="${prefix}_wheel_joint" type="continuous">
+            <parent link="base_link"/>
+            <child link="${prefix}_wheel"/>
+            <origin xyz="${x_pos} ${y_pos} 0" rpy="${-pi/2} 0 0" />
+            <axis xyz="0 0 1"/>
+        </joint>
+        <link name="${prefix}_wheel">
+            <visual>
+                <geometry>
+                    <cylinder radius="${wheel_radius}" length="${wheel_thickness}"/>
+                </geometry>
+                <material name="blue"/>
+            </visual>
+            <collision>
+                <geometry>
+                    <sphere radius="${wheel_radius}"/>
+                </geometry>
+            </collision>
+            <xacro:inertial_cylinder mass="${wheel_mass}" length="${wheel_thickness}" radius="${wheel_radius}">
+                <origin xyz="0 0 0" rpy="0 0 0"/>
+            </xacro:inertial_cylinder>
+        </link>
+    </xacro:macro>
+    <!-- Roues avant -->
+    <xacro:wheel prefix="front_left" x_pos="${wheel_offset_x_front}" y_pos="${wheel_offset_y}"/>
+    <xacro:wheel prefix="front_right" x_pos="${wheel_offset_x_front}" y_pos="${-wheel_offset_y}"/>
+    <!-- Roues arrière -->
+    <xacro:wheel prefix="rear_left" x_pos="${wheel_offset_x_rear}" y_pos="${wheel_offset_y}"/>
+    <xacro:wheel prefix="rear_right" x_pos="${wheel_offset_x_rear}" y_pos="${-wheel_offset_y}"/>
 </robot>
