Commit message: config de ros2_control

File: my_pkg/description/imu.xacro (robot description, xacro)
@@ -1,24 +1,2 @@
-<!--
-<?xml version="1.0"?>
-<robot xmlns:xacro="http://www.ros.org/wiki/xacro">
-    <joint name="imu_joint" type="fixed">
-            <origin xyz="0 0 0" rpy="0 0 0" />
-            <parent link="chassis"/>
-            <child link="imu_link" />
-    </joint>
-    <link name="imu_link">
-    </link>
-  <! Le pluging de l'imu >  commentaire
-    <gazebo reference= 'imu_link'>
-        <sensor name=' imu' type='imu'>
-            <always_on>1</always_on>
-            <update_rate>50</update_rate>
-            <visualize>true</visualize>
-            <topic>imu</topic>
-            <enable_metrics>true</enable_metrics>
-            <frame_id>imu_link</frame_id>
-        </sensor>
-    </gazebo>
-</robot>   -->
 <?xml version="1.0"?>
 <robot xmlns:xacro="http://www.ros.org/wiki/xacro" >
@@ -100,2 +78,24 @@
   </gazebo>
 </robot>
+<!--
+<?xml version="1.0"?>
+<robot xmlns:xacro="http://www.ros.org/wiki/xacro">
+    <joint name="imu_joint" type="fixed">
+            <origin xyz="0 0 0" rpy="0 0 0" />
+            <parent link="chassis"/>
+            <child link="imu_link" />
+    </joint>
+    <link name="imu_link">
+    </link>
+  <! Le pluging de l'imu >  commentaire
+    <gazebo reference= 'imu_link'>
+        <sensor name=' imu' type='imu'>
+            <always_on>1</always_on>
+            <update_rate>50</update_rate>
+            <visualize>true</visualize>
+            <topic>imu</topic>
+            <enable_metrics>true</enable_metrics>
+            <frame_id>imu_link</frame_id>
+        </sensor>
+    </gazebo>
+</robot>   -->

File: my_pkg/description/odom.xacro (robot description, xacro)
@@ -3,5 +3,5 @@
   <gazebo >
     <plugin filename="gz-sim-odometry-publisher-system" name="gz::sim::systems::OdometryPublisher">
-     <odom_topic>/odom </odom_topic>
+     <odom_topic>/odom</odom_topic>
      <odom_frame>odom</odom_frame>
     <robot_base_frame>base_footprint</robot_base_frame>

File: my_pkg/description/robot.urdf.xacro (robot description, xacro)
@@ -6,6 +6,6 @@
      <xacro:include filename="gps.xacro" />
      <xacro:include filename="odom.xacro" />
-      <xacro:include filename="ros2_control.xacro" />
-    <xacro:include filename="controle_gazebo.xacro" />
+     <xacro:include filename="ros2_control.xacro" />
+    <!--<xacro:include filename="controle_gazebo.xacro" /> -->
      <!-- Imu -->
      <xacro:include filename='imu.xacro'/>

File: my_pkg/description/robot.xacro (robot description, xacro)
@@ -31,5 +31,5 @@
         <color rgba="1 0 0 1"/>
     </material>
-    <link name="base_link">
+    <link name="base_footprint">
     </link>
     <joint name="base_footprint_joint" type="fixed">
@@ -38,5 +38,5 @@
         <origin xyz="0 0 ${wheel_radius}" rpy="0 0 0"/>
     </joint>
-    <link name="base_footprint">
+    <link name="base_link">
     </link>
     <joint name="chassis_joint" type="fixed">

File: my_pkg/description/ros2_control.xacro (robot description, xacro)
@@ -46,6 +46,6 @@
         <robot_param>robot_description</robot_param>
         <robot_param_node>robot_state_publisher</robot_param_node>
-        <parameters>$(my_pkg)/configuration/differentiel_controller.yaml</parameters>
-        <parameters>$(my_pkg)/configuration/gaz_ros2_ctl_use_sim.yaml</parameters>
+        <parameters>$(find my_pkg)/configuration/differentiel_controller.yaml</parameters>
+        <parameters>$(find my_pkg)/configuration/gaz_ros2_ctl_use_sim.yaml</parameters>
     </plugin>
   </gazebo>
